File: comp-btm.sch (EAGLE design)
At the start: 56 parts, among them IC1 LM358D, IC2 NE5532D, X1 POWER, X3 AUDIO

Commit message: V1 build
Parts:
- removed R26: 330k, rcl:R-EU_R0805
- removed R28: 1k, rcl:R-EU_R0805
- removed R29: 0R, rcl:R-EU_R0805
- removed R33: 100R, rcl:R-EU_R0805
- added C7: 470pF, rcl:C-EUC0805
- added R21: 1k, rcl:R-EU_R0805
- added R22: 47k, rcl:R-EU_R0805
- C1, C13: value 10uF -> NF; device rcl:CPOL-EUE3.5-8 -> rcl:C-EUC0805
- C10: device rcl:CPOL-EUE3.5-8 -> rcl:CPOL-EUE2,5-6E
- C11: value NF -> 1uF
- C12: value 1uF -> 10uF; device rcl:C-EUC0805 -> rcl:CPOL-EUE2,5-6E
- C14: value 1nF -> 470pF
- C15: value 1nF -> 10uF; device rcl:C-EUC0805 -> rcl:CPOL-EUE2,5-6E
- C2, C3: value 100nF -> 10uF; device rcl:C-EUC0805 -> rcl:CPOL-EUE2,5-6E
- C4: value 10uF -> 470pF; device rcl:CPOL-EUE3.5-8 -> rcl:C-EUC0805
- C5: value NF -> 100nF
- C6: value 470pF -> 100nF
- C8, C9: value 470pF -> 10nF
- R1: value 10k -> 1k
- R10: value 1k -> 47k
- R11, R23: value 100R -> NF; device rcl:R-EU_R0805 -> rcl:R-EU_0309/V
- R12: value NF -> 390R
- R14, R8: value 47k -> 1k
- R15: value 1M -> NF; device pot:TRIM_EU-B64Y -> rcl:R-EU_0309/V
- R16, R18, R19: value 0R -> 100R
- R20: value 0R -> NF
- R24: value NF -> 100R; device rcl:R-EU_0309/V -> rcl:R-EU_R0805
- R25: value 0R -> 330k
- R3: value 330k -> 10k
- R4, R5: value 1k -> 330k
- R7: value 1k -> 0R
- R9: value 390R -> 1k
- ZD1: value (none) -> 3V
- renumbered + to TP2, +1 to TP1, - to TP4, -1 to TP3, X3 to X2
Connections:
- removed net N$22: C11.1, J1.1, R1.1, R3.1, ZD1.C
- removed net OUTPUT_INV: C13.-, X2-3.S
- new net N$13: C15.+, R24.1
- new net OUTPUT_LPF: C12.-, X2-3.S
- net CTRL: now also R6.1; no longer R4.1
- net GND: now also C1.2, C2.-, C3.-, C4.2, C5.2, C6.2, C8.2, R2.1, R8.1, R9.1; no longer C1.-, C10.-, C11.2, C14.2, C2.2, C3.2, C9.2, R28.1, R6.1, R7.1
- net INPUT: now also C10.-; no longer C4.-
- net LED_GND: now also C11.2; no longer C12.2
- net N$1: now also R1.1, R2.2; no longer R5.1, R6.2
- net N$10: now also R11.2, R12.1; no longer R24.2, R9.1
- net N$11: now also C8.1, C9.1, R13.1, R14.2; no longer C14.1, C15.1, R10.2, R2.1
- net N$12: now also C4.1, IC1A.+IN, R4.1, R5.2, R6.2, R8.2; no longer R14.1, R15.A, R20.1
- net N$14: now also R7.2; no longer R18.2
- net N$15: now also J1.3, R25.2; no longer R15.S, R19.1, R20.2
- net N$17: now also C9.2, R16.2; no longer C15.2, R16.1, R33.2
- net N$18: now also R19.1; no longer R23.1
- net N$19: now also R23.1; no longer R29.1
- net N$2: now also C7.2, R10.2, R9.2; no longer C8.2, R7.2, R8.2
- net N$20: now also C11.1, R19.2; no longer C12.1, R23.2
- net N$21: now also R14.1; no longer R10.1
- net N$3: now also J1.1, R5.1; no longer C9.1, IC1A.+IN, R26.1, R28.2, R3.2, R4.2
- net N$4: now also C14.2, R15.2, R21.2, R22.2; no longer C6.2, R13.2, R14.2
- net N$5: now also C12.+, R16.1; no longer C13.+, R33.1
- net N$6: now also C7.1, R10.1, R11.1, R12.2; no longer C8.1, R24.1, R8.1, R9.2
- net N$7: now also C13.1, R18.2, R20.2; no longer C5.1, R11.2, R12.2
- net N$8: now also C10.+, R18.1; no longer C4.+, R11.1
- net N$9: now also C1.1, R3.1, R4.2, ZD1.C; no longer R26.2
- net OUTPUT: now also C15.-
- net V2: now also C13.2, C3.+, R20.1, R21.1, R7.1; no longer C10.+, C5.2, R12.1, R13.1, R18.1
- net VCC: now also C2.+, C5.1, C6.1, R3.2; no longer C1.+, C2.1, C3.1, R5.2
- net V_OUT: now also C14.1, R13.2, R15.1, R22.1, R23.2, R24.2; no longer C6.1, R15.E, R16.2, R19.2, R2.2, R25.2, R29.2
Other:
- moved on the sheet: C10, C11, C14, C5, C6, C8, C9, D1, D2, R1, R10, R11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
